File: zglue-jade-adapter.sch (KiCad schematic (older format))
At the start: 77 parts, among them J1 543630489, J2 543630489, U1 zGlue-Jade

Commit message: Regenerate libraries
Parts:
- C1: footprint antmicro-footprints:0402-cap -> zglue-jade-adapter-footprints:0402-cap; symbol antmicroCapacitors0402:C_10u_0402 -> zglue-jade-adapter:C_10u_0402
- C10, C14, C5, C6, C7, C9: footprint antmicro-footprints:0402-cap -> zglue-jade-adapter-footprints:0402-cap; symbol antmicroCapacitors0402:C_100n_0402_6V3 -> zglue-jade-adapter:C_100n_0402_6V3
- C11: footprint antmicro-footprints:0603-cap -> zglue-jade-adapter-footprints:0603-cap; symbol antmicroCapacitors0603:C_1u_0603 -> zglue-jade-adapter:C_1u_0603
- C15: footprint antmicro-footprints:0402-cap -> zglue-jade-adapter-footprints:0402-cap; symbol antmicroCapacitors0402:C_10n_0402 -> zglue-jade-adapter:C_10n_0402
- C2, C3, C4: footprint antmicro-footprints:0402-cap -> zglue-jade-adapter-footprints:0402-cap; symbol antmicroCapacitors0402:C_2u2_0402 -> zglue-jade-adapter:C_2u2_0402
- J1, J2: footprint antmicro-footprints:543630489 -> zglue-jade-adapter-footprints:543630489; symbol antmicroB2bConnectors:543630489 -> zglue-jade-adapter:543630489; MPN (none) -> 543630489; Manufacturer (none) -> Molex
- R1, R15, R16, R17, R18, R19, R2, R20, R21, R22, R29, R3, R4, R5, R6, R7, R8: footprint antmicro-footprints:0402-res -> zglue-jade-adapter-footprints:0402-res; symbol antmicroResistors0402:R_0R_0402 -> zglue-jade-adapter:R_0R_0402
- R10: footprint antmicro-footprints:0402-res -> zglue-jade-adapter-footprints:0402-res; symbol antmicroResistors0402:R_220R_0402 -> zglue-jade-adapter:R_220R_0402
- R11: footprint antmicro-footprints:0402-res -> zglue-jade-adapter-footprints:0402-res; symbol antmicroResistors0402:R_1k5_0402 -> zglue-jade-adapter:R_1k5_0402
- R12, R13, R28, R9: footprint antmicro-footprints:0402-res -> zglue-jade-adapter-footprints:0402-res; symbol antmicroResistors0402:R_100R_0402 -> zglue-jade-adapter:R_100R_0402
- R14, R25, R30, R31: footprint antmicro-footprints:0402-res -> zglue-jade-adapter-footprints:0402-res; symbol antmicroResistors0402:R_22R_0402 -> zglue-jade-adapter:R_22R_0402
- R23, R24: footprint antmicro-footprints:0402-res -> zglue-jade-adapter-footprints:0402-res; symbol antmicroResistors0402:R_100R_0402 -> zglue-jade-adapter:R_100R_0402; MPN (none) -> CR0402-FX-1000GLF; Manufacturer (none) -> BOURNS; Val 120R -> 100R
- R26, R27: footprint antmicro-footprints:0402-res -> zglue-jade-adapter-footprints:0402-res; symbol antmicroResistors0402:R_49R9_0402 -> zglue-jade-adapter:R_49R9_0402
- TP1, TP10, TP11, TP12, TP13, TP14, TP15, TP16, TP17, TP18, TP19, TP20, TP21, TP22, TP23, TP24, TP25, TP26, TP27, TP29, TP3, TP32, TP33, TP34, TP35, TP4, TP5, TP6, TP7, TP8, TP9: footprint antmicro-footprints:Testpoint_smd_1mm -> zglue-jade-adapter-footprints:Testpoint_smd_1mm; symbol antmicroTestPoints:TP_SMD1MM -> zglue-jade-adapter:TP_SMD1MM
- U1: footprint lib:Z-Glue_LGA-96 -> zglue-jade-adapter-footprints:Z-Glue_LGA-96; symbol zglue-jade-adapter-rescue:zGlue-Jade-zglue-jade -> zglue-jade-adapter:zGlue-Jade-zglue-jade
