File: zglue-gem2-adapter.kicad_pcb (KiCad board)
At the start: 6 copper layers, 25 x 20 mm, 77 parts, among them J1 543630489, J2 543630489, U1 zGlue-Jade

Commit message: Update PCB
Parts:
- U1: value zGlue-Jade -> GEM2
Changed lines of the file:
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@@
-(kicad_pcb (version 20171130) (host pcbnew 5.1.5)
+(kicad_pcb (version 20171130) (host pcbnew 5.1.5+dfsg1-2~bpo10+1)
   (general
     (thickness 1)
@@
       (effects (font (size 0.7 0.7) (thickness 0.15)))
     )
-    (fp_text value zGlue-Jade (at 0 7.475) (layer F.Fab)
+    (fp_text value GEM2 (at 0 7.475) (layer F.Fab)
       (effects (font (size 1 1) (thickness 0.15)))
     )
