File: gem2-adapter.sch (KiCad schematic (older format))
At the start: 77 parts, among them J1 543630489, J2 543630489, U1 GEM2

Commit message: Update library naming
Parts:
- C1: footprint zglue-jade-adapter-footprints:0402-cap -> gem2-adapter-footprints:0402-cap; symbol zglue-jade-adapter:C_10u_0402 -> gem2-adapter:C_10u_0402
- C10, C14, C5, C6, C7, C9: footprint zglue-jade-adapter-footprints:0402-cap -> gem2-adapter-footprints:0402-cap; symbol zglue-jade-adapter:C_100n_0402_6V3 -> gem2-adapter:C_100n_0402_6V3
- C11: footprint zglue-jade-adapter-footprints:0603-cap -> gem2-adapter-footprints:0603-cap; symbol zglue-jade-adapter:C_1u_0603 -> gem2-adapter:C_1u_0603
- C15: footprint zglue-jade-adapter-footprints:0402-cap -> gem2-adapter-footprints:0402-cap; symbol zglue-jade-adapter:C_10n_0402 -> gem2-adapter:C_10n_0402
- C2, C3, C4: footprint zglue-jade-adapter-footprints:0402-cap -> gem2-adapter-footprints:0402-cap; symbol zglue-jade-adapter:C_2u2_0402 -> gem2-adapter:C_2u2_0402
- J1, J2: footprint zglue-jade-adapter-footprints:543630489 -> gem2-adapter-footprints:543630489; symbol zglue-jade-adapter:543630489 -> gem2-adapter:543630489
- R1, R15, R16, R17, R18, R19, R2, R20, R21, R22, R29, R3, R4, R5, R6, R7, R8: footprint zglue-jade-adapter-footprints:0402-res -> gem2-adapter-footprints:0402-res; symbol zglue-jade-adapter:R_0R_0402 -> gem2-adapter:R_0R_0402
- R10: footprint zglue-jade-adapter-footprints:0402-res -> gem2-adapter-footprints:0402-res; symbol zglue-jade-adapter:R_220R_0402 -> gem2-adapter:R_220R_0402
- R11: footprint zglue-jade-adapter-footprints:0402-res -> gem2-adapter-footprints:0402-res; symbol zglue-jade-adapter:R_1k5_0402 -> gem2-adapter:R_1k5_0402
- R12, R13, R23, R24, R28, R9: footprint zglue-jade-adapter-footprints:0402-res -> gem2-adapter-footprints:0402-res; symbol zglue-jade-adapter:R_100R_0402 -> gem2-adapter:R_100R_0402
- R14, R25, R30, R31: footprint zglue-jade-adapter-footprints:0402-res -> gem2-adapter-footprints:0402-res; symbol zglue-jade-adapter:R_22R_0402 -> gem2-adapter:R_22R_0402
- R26, R27: footprint zglue-jade-adapter-footprints:0402-res -> gem2-adapter-footprints:0402-res; symbol zglue-jade-adapter:R_49R9_0402 -> gem2-adapter:R_49R9_0402
- TP1, TP10, TP11, TP12, TP13, TP14, TP15, TP16, TP17, TP18, TP19, TP20, TP21, TP22, TP23, TP24, TP25, TP26, TP27, TP29, TP3, TP32, TP33, TP34, TP35, TP4, TP5, TP6, TP7, TP8, TP9: footprint zglue-jade-adapter-footprints:Testpoint_smd_1mm -> gem2-adapter-footprints:Testpoint_smd_1mm; symbol zglue-jade-adapter:TP_SMD1MM -> gem2-adapter:TP_SMD1MM
- U1: footprint zglue-jade-adapter-footprints:Z-Glue_LGA-96 -> gem2-adapter-footprints:Z-Glue_LGA-96; symbol zglue-jade-adapter:GEM2 -> gem2-adapter:GEM2
